File: JosEffigy-Keymix-Basic.kicad_pcb (KiCad board)
At the start: 2 copper layers, 177.8 x 120.6 mm, 25 parts, among them U1 Pico

Commit message: 1.1
Parts:
- renumbered MX5 to HOME, MX6 to SELECT, MX7 to START
Routing:
- net 3K: track 147.2 -> 165.4 mm, vias 1 -> 0
- net 1K: track 79.6 -> 81.9 mm, vias 0 -> 1
- net 4P: track 92.5 -> 94.5 mm
- net LEFT: track 147.9 -> 149.5 mm, vias 1 -> 2
- net RIGHT: track 87.1 -> 88.7 mm
- net 2K: track 89.0 -> 90.4 mm, vias 0 -> 1
- net UP: track 171.2 -> 170.2 mm, vias 0 -> 1
- net 4K: track 169.1 -> 170.0 mm
- added copper zone on F.Cu, net (none)
Other:
- board text removed: "Home"
- board text removed: "Select"
- board text removed: "Start"

Commit message: 1.2
Added center mounting hole
Parts:
- added h1: MountingHole_3.5mm, MountingHole:MountingHole_3.5mm, F.Cu at (150.0, 96.8)
Changed lines of the file:
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@@
       (net 14 "3P") (pinfunction "ROW") (pintype "passive"))
+  )
+  (footprint "MountingHole:MountingHole_3.5mm" (layer "F.Cu")
+    (at 150.01875 96.8375)
+    (descr "Mounting Hole 3.5mm, no annular")
+    (tags "mounting hole 3.5mm no annular")
+    (attr board_only exclude_from_pos_files exclude_from_bom)
+    (fp_text reference "h1" (at 0 -4.5) (layer "F.SilkS") hide
+        (effects (font (size 1 1) (thickness 0.15)))
+    )
+    (fp_text value "MountingHole_3.5mm" (at 0 4.5) (layer "F.Fab")
+        (effects (font (size 1 1) (thickness 0.15)))
+    )
+    (fp_text user "${REFERENCE}" (at 0 0) (layer "F.Fab")
+        (effects (font (size 1 1) (thickness 0.15)))
+    )
+    (fp_circle (center 0 0) (end 3.5 0)
+      (stroke (width 0.15) (type solid)) (fill none) (layer "Cmts.User"))
+    (fp_circle (center 0 0) (end 3.75 0)
+      (stroke (width 0.05) (type solid)) (fill none) (layer "F.CrtYd"))
+    (pad "" np_thru_hole circle (at 0 0) (size 3.5 3.5) (drill 3.5) (layers "F&B.Cu" "*.Mask"))
   )
   (footprint "keyswitches:Kailh_socket_MX_optional" (layer "F.Cu")
